File: LEDs.kicad_sch (KiCad schematic)
At the start: 10 parts

Commit message: more lights
Parts:
- added C36, C37, C38, C39: 1uF, Capacitor_SMD:C_0603_1608Metric, symbol Device:C
- added WLED6, WLED7, WLED8, WLED9: WS2812B, LED_SMD:LED_WS2812B_PLCC4_5.0x5.0mm_P3.2mm, symbol LED:WS2812B
Connections:
- net GND: now also C36.2, C37.2, C38.2, C39.2, WLED6.3 (VSS), WLED7.3 (VSS), WLED8.3 (VSS), WLED9.3 (VSS)
- net VBAT: now also C36.1, C37.1, C38.1, C39.1, WLED6.1 (VDD), WLED7.1 (VDD), WLED8.1 (VDD), WLED9.1 (VDD)
- net at WLED5.2 (DOUT): now also WLED6.4 (DIN)
- new net: WLED7.2 (DOUT), WLED8.4 (DIN)
- new net: WLED6.2 (DOUT), WLED7.4 (DIN)
- new net: WLED8.2 (DOUT), WLED9.4 (DIN)
