File: fiona-the-rat.kicad_pcb (KiCad board)
At the start: 2 copper layers, 83.3 x 89.9 mm, 96 parts, among them J1 USB_TP_P, J10 ~{CHG}_TP, J11 +1V1_TP, J12 VBAT_TP, J13 +3V3_TP, J14 SWD, J15 BMS_COUT_TP, J16 BMS_DOUT_TP, J17 BAT_P_JMP, J18 BAT_N_JMP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

Commit message: more lights
Parts:
- added C36: 1uF, Capacitor_SMD:C_0603_1608Metric, F.Cu at (130.3, 125.0)
- added C37: 1uF, Capacitor_SMD:C_0603_1608Metric, F.Cu at (130.3, 133.1)
- added C38: 1uF, Capacitor_SMD:C_0603_1608Metric, F.Cu at (149.1, 133.1)
- added C39: 1uF, Capacitor_SMD:C_0603_1608Metric, F.Cu at (149.1, 125.0)
- added WLED6: WS2812B, LED_SMD:LED_WS2812B_PLCC4_5.0x5.0mm_P3.2mm, F.Cu at (130.3, 121.4)
- added WLED7: WS2812B, LED_SMD:LED_WS2812B_PLCC4_5.0x5.0mm_P3.2mm, F.Cu at (130.3, 136.7)
- added WLED8: WS2812B, LED_SMD:LED_WS2812B_PLCC4_5.0x5.0mm_P3.2mm, F.Cu at (149.1, 136.7)
- added WLED9: WS2812B, LED_SMD:LED_WS2812B_PLCC4_5.0x5.0mm_P3.2mm, F.Cu at (149.1, 121.4)
Routing:
- net VBAT: track 290.6 -> 365.5 mm
- net Net-(WLED5-DOUT): track 0.00 -> 61.4 mm, vias 0 -> 4
- net Net-(WLED7-DOUT): track 0.00 -> 25.8 mm
- net Net-(WLED8-DOUT): track 0.00 -> 20.6 mm
- net Net-(WLED6-DOUT): track 0.00 -> 15.5 mm
- net GND: track 122.4 -> 125.7 mm, vias 98 -> 103
- net /UI_buttons/SW_R: track 35.1 -> 35.9 mm

Commit message: Update fiona-the-rat.kicad_pcb
add 0.0.2 text
Other:
- board text added: "0.0.2"
Changed lines of the file:
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@@
+		)
+	)
+	(gr_text "0.0.2"
+		(at 99.822 74.422 0)
+		(layer "F.SilkS")
+		(effects
+			(font
+				(size 2.032 2.032)
+				(thickness 0.3048)
+				(bold yes)
+			)
+			(justify left bottom)
 		)
 	)
@@
 		)
 	)
+	(gr_text "0.0.2"
+		(at 107.95 74.422 -0)
+		(layer "B.SilkS")
+		(effects
+			(font
+				(size 2.032 2.032)
+				(thickness 0.3048)
+				(bold yes)
+			)
+			(justify left bottom mirror)
+		)
+	)

Commit message: changed lib to owned
Parts:
- BT1: footprint 1043P:BAT_1043P -> pfornage-kicad-lib:BAT_1043P
- C25: value 0.1uF -> 100nF
- MOSFET1: footprint DMN3042L-7-footprints:SOT23_DMN3042L_DIO -> pfornage-kicad-lib:SOT23_DMN3042L_DIO
- R11: value 2.2k -> 2.2K
- R8: value 1k -> 1K
- SW1: footprint 1825027_8:SW2_1825027-C_TEC -> pfornage-kicad-lib:SW2_1825027-C_TEC
- SW2: footprint OS102011MA1QN1:OS102011MA1QN1_CNK -> pfornage-kicad-lib:OS102011MA1QN1_CNK
- SW_D1, SW_E1, SW_L1, SW_R1, SW_U1: footprint 1825910_6:SW_1825910-6-4 -> pfornage-kicad-lib:SW_1825910-6-4
- U2: footprint Adafruit-1.3-inch-display:display -> pfornage-kicad-lib:adafruit-4313-display
- U3: footprint W25Q128JVSIQ:SOIC127P790X216-8N -> pfornage-kicad-lib:SOIC127P790X216-8N
- U4: footprint BQ21040DBVR:SOT95P280X145-6N -> pfornage-kicad-lib:SOT95P280X145-6N
- U6, U7: footprint CSD16406Q3:TRANS_CSD16406Q3 -> pfornage-kicad-lib:TRANS_CSD16406Q3
- U8: footprint BQ29700DSER:SON50P150X150X80-6N -> pfornage-kicad-lib:SON50P150X150X80-6N
