File: UI_buttons.kicad_sch (KiCad schematic)
At the start: 10 parts

Commit message: change lib to owned
Parts:
- SW_D1, SW_E1, SW_L1, SW_R1, SW_U1: footprint 1825910_6:SW_1825910-6-4 -> pfornage-kicad-lib:SW_1825910-6-4; symbol 1825910-6:1825910-6 -> pfornage-kicad-lib:1825910-6
Changed lines of the file:
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@@
 	)
 	(symbol
-		(lib_id "1825910-6:1825910-6")
+		(lib_id "pfornage-kicad-lib:1825910-6")
 		(at 151.13 105.41 0)
 		(unit 1)
@@
 			)
 		)
-		(property "Footprint" "1825910_6:SW_1825910-6-4"
+		(property "Footprint" "pfornage-kicad-lib:SW_1825910-6-4"
 			(at 151.13 105.41 0)
 			(effects
@@
 	)
 	(symbol
-		(lib_id "1825910-6:1825910-6")
+		(lib_id "pfornage-kicad-lib:1825910-6")
 		(at 125.73 120.65 0)
 		(unit 1)
@@
 			)
 		)
-		(property "Footprint" "1825910_6:SW_1825910-6-4"
+		(property "Footprint" "pfornage-kicad-lib:SW_1825910-6-4"
 			(at 125.73 120.65 0)
 			(effects
@@
 	)
 	(symbol
-		(lib_id "1825910-6:1825910-6")
+		(lib_id "pfornage-kicad-lib:1825910-6")
 		(at 125.73 105.41 0)
 		(unit 1)
@@
 			)
 		)
-		(property "Footprint" "1825910_6:SW_1825910-6-4"
+		(property "Footprint" "pfornage-kicad-lib:SW_1825910-6-4"
 			(at 125.73 105.41 0)
 			(effects
@@
 	)
 	(symbol
-		(lib_id "1825910-6:1825910-6")
+		(lib_id "pfornage-kicad-lib:1825910-6")
 		(at 125.73 90.17 0)
 		(unit 1)
@@
 			)
 		)
-		(property "Footprint" "1825910_6:SW_1825910-6-4"
+		(property "Footprint" "pfornage-kicad-lib:SW_1825910-6-4"
 			(at 125.73 90.17 0)
 			(effects
@@
 	)
 	(symbol
-		(lib_id "1825910-6:1825910-6")
+		(lib_id "pfornage-kicad-lib:1825910-6")
 		(at 95.25 105.41 0)
 		(unit 1)
@@
 			)
 		)
-		(property "Footprint" "1825910_6:SW_1825910-6-4"
+		(property "Footprint" "pfornage-kicad-lib:SW_1825910-6-4"
 			(at 95.25 105.41 0)
 			(effects
