File: pack.kicad_sch (KiCad schematic)
At the start: 15 parts, among them J10 BMS_COUT_TP, J11 BMS_DOUT_TP, J12 BAT_P_JMP, J13 BAT_N_JMP, SW2 OS102011MA1QN1, U6 CSD16406Q3, U7 CSD16406Q3, U8 BQ29700DSER

Commit message: adding stuff
Parts:
- renumbered J10 to J15, J11 to J16, J12 to J17, J13 to J18, R10 to R11, R11 to R12, R12 to R13, R13 to R14
Changed lines of the file:
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@@
 		(on_board yes)
 		(dnp no)
-		(property "Reference" "J12"
+		(property "Reference" "J17"
 			(at 202.565 74.93 0)
 			(effects
@@
 			(project "fiona-the-rat"
 				(path "/43ed14e6-1321-4146-9b65-20c47dea76d8/c3eec74b-c069-43e1-91b8-c99de172a1b4"
-					(reference "J12")
+					(reference "J17")
 					(unit 1)
 				)
@@
 		(on_board yes)
 		(dnp no)
-		(property "Reference" "R10"
+		(property "Reference" "R11"
 			(at 88.138 108.7119 0)
 			(effects
@@
 			(project "fiona-the-rat"
 				(path "/43ed14e6-1321-4146-9b65-20c47dea76d8/c3eec74b-c069-43e1-91b8-c99de172a1b4"
-					(reference "R10")
+					(reference "R11")
 					(unit 1)
 				)
@@
 		(on_board yes)
 		(dnp no)
-		(property "Reference" "J13"
+		(property "Reference" "J18"
 			(at 202.565 86.36 0)
 			(effects
@@
 			(project "fiona-the-rat"
 				(path "/43ed14e6-1321-4146-9b65-20c47dea76d8/c3eec74b-c069-43e1-91b8-c99de172a1b4"
-					(reference "J13")
+					(reference "J18")
 					(unit 1)
 				)
@@
 		(on_board yes)
 		(dnp no)
-		(property "Reference" "R12"
+		(property "Reference" "R13"
 			(at 150.622 112.5219 90)
 			(effects
@@
 			(project "fiona-the-rat"
 				(path "/43ed14e6-1321-4146-9b65-20c47dea76d8/c3eec74b-c069-43e1-91b8-c99de172a1b4"
-					(reference "R12")
+					(reference "R13")
 					(unit 1)
 				)
@@
 		(on_board yes)
 		(dnp no)
-		(property "Reference" "J11"
+		(property "Reference" "J16"
 			(at 109.855 80.01 0)
 			(effects
@@
 			(project "fiona-the-rat"
 				(path "/43ed14e6-1321-4146-9b65-20c47dea76d8/c3eec74b-c069-43e1-91b8-c99de172a1b4"
-					(reference "J11")
+					(reference "J16")
 					(unit 1)
 				)
@@
 		(dnp no)
 		(fields_autoplaced yes)
-		(property "Reference" "R13"
+		(property "Reference" "R14"
 			(at 167.64 67.3099 0)
 			(effects
@@
 			(project "fiona-the-rat"
 				(path "/43ed14e6-1321-4146-9b65-20c47dea76d8/c3eec74b-c069-43e1-91b8-c99de172a1b4"
-					(reference "R13")
+					(reference "R14")
 					(unit 1)
 				)
@@
 		(on_board yes)
 		(dnp no)
-		(property "Reference" "J10"
+		(property "Reference" "J15"
 			(at 109.855 76.2 0)
 			(effects
@@
 			(project "fiona-the-rat"
 				(path "/43ed14e6-1321-4146-9b65-20c47dea76d8/c3eec74b-c069-43e1-91b8-c99de172a1b4"
-					(reference "J10")
+					(reference "J15")
 					(unit 1)
 				)
@@
 		(on_board yes)
 		(dnp no)
-		(property "Reference" "R11"
+		(property "Reference" "R12"
 			(at 98.298 112.5219 90)
 			(effects
@@
 			(project "fiona-the-rat"
 				(path "/43ed14e6-1321-4146-9b65-20c47dea76d8/c3eec74b-c069-43e1-91b8-c99de172a1b4"
-					(reference "R11")
+					(reference "R12")
 					(unit 1)
 				)

Commit message: change lib to owned
Parts:
- BT1: footprint 1043P:BAT_1043P -> pfornage-kicad-lib:BAT_1043P; symbol 1043P:1043P -> pfornage-kicad-lib:1043P
- C25: value 0.1uF -> 100nF
- R11: value 2.2k -> 2.2K
- SW2: footprint OS102011MA1QN1_CNK -> pfornage-kicad-lib:OS102011MA1QN1_CNK; symbol 2025-07-08_19-42-59:OS102011MA1QN1 -> pfornage-kicad-lib:OS102011MA1QN1
- U6, U7: footprint CSD16406Q3:TRANS_CSD16406Q3 -> pfornage-kicad-lib:TRANS_CSD16406Q3; symbol CSD16406Q3:CSD16406Q3 -> pfornage-kicad-lib:CSD16406Q3
- U8: footprint BQ29700DSER:SON50P150X150X80-6N -> pfornage-kicad-lib:SON50P150X150X80-6N; symbol BQ29700DSER:BQ29700DSER -> pfornage-kicad-lib:BQ29700DSER
Changed lines of the file:
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@@
 	)
 	(symbol
-		(lib_id "2025-07-08_19-42-59:OS102011MA1QN1")
+		(lib_id "pfornage-kicad-lib:OS102011MA1QN1")
 		(at 109.22 81.28 90)
 		(mirror x)
@@
 			)
 		)
-		(property "Footprint" "OS102011MA1QN1_CNK"
+		(property "Footprint" "pfornage-kicad-lib:OS102011MA1QN1_CNK"
 			(at 109.22 81.28 0)
 			(effects
@@
 		(dnp no)
 		(property "Reference" "R11"
-			(at 88.138 108.7119 0)
+			(at 90.678 110.9979 90)
 			(effects
 				(font
@@
 			)
 		)
-		(property "Value" "2.2k"
-			(at 92.71 111.2519 90)
-			(effects
-				(font
-					(size 1.27 1.27)
-				)
-				(justify left)
+		(property "Value" "2.2K"
+			(at 92.71 109.2199 90)
+			(effects
+				(font
+					(size 1.27 1.27)
+				)
 			)
 		)
@@
 		(on_board yes)
 		(dnp no)
-		(fields_autoplaced yes)
 		(property "Reference" "R14"
-			(at 167.64 67.3099 0)
+			(at 167.386 70.6119 90)
 			(effects
 				(font
@@
 		)
 		(property "Value" "330"
-			(at 167.64 69.8499 0)
-			(effects
-				(font
-					(size 1.27 1.27)
-				)
-				(justify left)
+			(at 165.1 68.5799 90)
+			(effects
+				(font
+					(size 1.27 1.27)
+				)
 			)
 		)
@@
 	)
 	(symbol
-		(lib_id "CSD16406Q3:CSD16406Q3")
+		(lib_id "pfornage-kicad-lib:CSD16406Q3")
 		(at 113.03 114.3 0)
 		(mirror x)
@@
 			)
 		)
-		(property "Footprint" "CSD16406Q3:TRANS_CSD16406Q3"
+		(property "Footprint" "pfornage-kicad-lib:TRANS_CSD16406Q3"
 			(at 113.03 114.3 0)
 			(effects
@@
 			)
 		)
-		(property "Description" ""
+		(property "Description" "25V, N ch NexFET MOSFET, single SON3x3, 7.4mOhm 8-VSON-CLIP -55 to 150"
 			(at 113.03 114.3 0)
 			(effects
@@
 					(size 1.27 1.27)
 				)
+				(justify bottom)
 				(hide yes)
 			)
@@
 	)
 	(symbol
-		(lib_name "CSD16406Q3_1")
-		(lib_id "CSD16406Q3:CSD16406Q3")
+		(lib_id "pfornage-kicad-lib:CSD16406Q3")
 		(at 135.89 114.3 180)
 		(unit 1)
@@
 			)
 		)
-		(property "Footprint" "CSD16406Q3:TRANS_CSD16406Q3"
+		(property "Footprint" "pfornage-kicad-lib:TRANS_CSD16406Q3"
 			(at 135.89 114.3 0)
 			(effects
@@
 			)
 		)
-		(property "Description" ""
+		(property "Description" "25V, N ch NexFET MOSFET, single SON3x3, 7.4mOhm 8-VSON-CLIP -55 to 150"
 			(at 135.89 114.3 0)
 			(effects
@@
 					(size 1.27 1.27)
 				)
+				(justify bottom)
 				(hide yes)
 			)
@@
 	)
 	(symbol
-		(lib_id "1043P:1043P")
+		(lib_id "pfornage-kicad-lib:1043P")
 		(at 194.31 78.74 270)
 		(unit 1)
@@
 			)
 		)
-		(property "Footprint" "1043P:BAT_1043P"
+		(property "Footprint" "pfornage-kicad-lib:BAT_1043P"
 			(at 194.31 78.74 0)
 			(effects
@@
 	)
 	(symbol
-		(lib_id "BQ29700DSER:BQ29700DSER")
+		(lib_id "pfornage-kicad-lib:BQ29700DSER")
 		(at 143.51 83.82 0)
 		(mirror y)
@@
 			)
 		)
-		(property "Footprint" "BQ29700DSER:SON50P150X150X80-6N"
+		(property "Footprint" "pfornage-kicad-lib:SON50P150X150X80-6N"
 			(at 143.51 83.82 0)
 			(effects
@@
 			)
 		)
-		(property "Value" "0.1uF"
+		(property "Value" "100nF"
 			(at 168.91 88.8999 0)
 			(effects
